File: GSM Schematic.sch (EAGLE design)
At the start: 19 parts, among them IC1 7805T, J1 5.5x2.1mm Barrel, J2 AVR_SPI_PRG_62X3_LOCK, Q2 16M, U1 ATMEGA328P-PU

Commit message: Add files via upload
Parts:
- removed C2, C4: 10u, rcl:C-EUC0603
- removed LED1: (no value), led:LEDSML0603
- added C3, C5: 10u, rcl:CPOL-EUE5-10.5
- added LED3: (no value), led:LED5MM
Connections:
- removed net N$11: C4.1, IC1.VO, J2.2, R1.1, R3.2, U1.AREF, U1.AVCC
- removed net N$17: C2.1, DOORSTRIKE-2.KL, IC1.VI, J1.PWR, SPDT.NC
- new net 12V: C3.+, DOORSTRIKE-2.KL, IC1.VI, J1.PWR, SPDT.NC
- new net 5V: C5.+, IC1.VO, J2.2, R1.1, R3.2, U1.AREF, U1.AVCC
- net GND: now also C3.-, C5.-, LED3.C; no longer C2.2, C4.2, LED1.C
- net N$6: now also LED3.A; no longer LED1.A
Other:
- note added: "8"
- note added: "GSM SENSOR GROUP"
- note removed: "7"
Changed lines of the file:
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@@
 <?xml version="1.0" encoding="utf-8"?>
 <!DOCTYPE eagle SYSTEM "eagle.dtd">
-<eagle version="7.6.0">
+<eagle version="7.7.0">
 <drawing>
 <settings>
@@
 <setting verticaltext="up"/>
 </settings>
-<grid distance="0.1" unitdist="inch" unit="inch" style="lines" multiple="1" display="no" altdistance="0.01" altunitdist="inch" altunit="inch"/>
+<grid distance="0.05" unitdist="inch" unit="inch" style="lines" multiple="2" display="yes" altdistance="0.01" altunitdist="inch" altunit="inch"/>
 <layers>
 <layer number="1" name="Top" color="4" fill="1" visible="no" active="no"/>
@@
 <part name="R3" library="rcl" deviceset="R-US_" device="R0603" value="220"/>
 <part name="R1" library="rcl" deviceset="R-US_" device="R0603" value="10k"/>
-<part name="C4" library="rcl" deviceset="C-EU" device="C0603" value="10u"/>
-<part name="C2" library="rcl" deviceset="C-EU" device="C0603" value="10u"/>
 <part name="LED2" library="led" deviceset="LED" device="SML0603"/>
 <part name="J2" library="SparkFun-Connectors" deviceset="AVR_SPI_PRG_6" device="2X3_LOCK"/>
@@
 <part name="DOORSTRIKE" library="con-wago-500" deviceset="W237-102" device=""/>
 <part name="R2" library="rcl" deviceset="R-US_" device="R0603" value="220"/>
-<part name="LED1" library="led" deviceset="LED" device="SML0603"/>
 <part name="GND5" library="supply1" deviceset="GND" device=""/>
+<part name="C3" library="rcl" deviceset="CPOL-EU" device="E5-10.5" value="10u"/>
+<part name="C5" library="rcl" deviceset="CPOL-EU" device="E5-10.5" value="10u"/>
+<part name="LED3" library="led" deviceset="LED" device="5MM"/>
 </parts>
 <sheets>
 <sheet>
 <plain>
-<text x="330.2" y="7.62" size="1.778" layer="91">1</text>
-<text x="419.1" y="7.62" size="1.778" layer="91">7</text>
+<text x="359.41" y="7.62" size="3.81" layer="97" font="vector">1</text>
+<text x="422.91" y="7.62" size="3.81" layer="97" font="vector">8</text>
+<text x="347.98" y="27.94" size="3.81" layer="97" font="vector">GSM SENSOR GROUP</text>
 </plain>
 <instances>
@@
 <attribute name="VALUE" x="204.47" y="174.498" size="1.778" layer="96"/>
 </instance>
-<instance part="C4" gate="G$1" x="187.96" y="203.2"/>
-<instance part="C2" gate="G$1" x="160.02" y="203.2"/>
 <instance part="LED2" gate="G$1" x="185.42" y="170.18" smashed="yes">
 <attribute name="NAME" x="181.102" y="169.926" size="1.778" layer="95" rot="R180"/>
@@
 <attribute name="VALUE" x="283.21" y="146.558" size="1.778" layer="96"/>
 </instance>
-<instance part="LED1" gate="G$1" x="297.18" y="149.86" smashed="yes" rot="R90">
-<attribute name="NAME" x="297.434" y="158.242" size="1.778" layer="95" rot="R270"/>
-<attribute name="VALUE" x="301.752" y="155.575" size="1.778" layer="96" rot="R180"/>
-</instance>
-<instance part="GND5" gate="1" x="304.8" y="146.05" smashed="yes">
-<attribute name="VALUE" x="302.26" y="143.51" size="1.778" layer="96"/>
-</instance>
+<instance part="GND5" gate="1" x="314.96" y="144.78" smashed="yes">
+<attribute name="VALUE" x="312.42" y="142.24" size="1.778" layer="96"/>
+</instance>
+<instance part="C3" gate="G$1" x="160.02" y="203.2"/>
+<instance part="C5" gate="G$1" x="187.96" y="203.2"/>
+<instance part="LED3" gate="G$1" x="295.91" y="149.86" rot="R90"/>
 </instances>
 <busses>
@@
 <wire x1="160.02" y1="195.58" x2="175.26" y2="195.58" width="0.1524" layer="91"/>
 <junction x="175.26" y="195.58"/>
-<pinref part="C2" gate="G$1" pin="2"/>
+<pinref part="C3" gate="G$1" pin="-"/>
 </segment>
 <segment>
@@
 <segment>
 <pinref part="GND3" gate="1" pin="GND"/>
-<pinref part="C4" gate="G$1" pin="2"/>
 <wire x1="187.96" y1="198.12" x2="187.96" y2="195.58" width="0.1524" layer="91"/>
+<pinref part="C5" gate="G$1" pin="-"/>
 </segment>
 <segment>
@@
 </segment>
 <segment>
-<pinref part="LED1" gate="G$1" pin="C"/>
-<wire x1="302.26" y1="149.86" x2="304.8" y2="149.86" width="0.1524" layer="91"/>
-<wire x1="304.8" y1="149.86" x2="304.8" y2="148.59" width="0.1524" layer="91"/>
+<wire x1="300.99" y1="149.86" x2="314.96" y2="149.86" width="0.1524" layer="91"/>
+<wire x1="314.96" y1="149.86" x2="314.96" y2="147.32" width="0.1524" layer="91"/>
 <pinref part="GND5" gate="1" pin="GND"/>
+<pinref part="LED3" gate="G$1" pin="C"/>
 </segment>
 </net>
@@
 </segment>
 </net>
-<net name="N$11" class="0">
+<net name="5V" class="0">
 <segment>
 <pinref part="IC1" gate="A1" pin="VO"/>
@@
 <junction x="195.58" y="177.8"/>
 <pinref part="R1" gate="G$1" pin="1"/>
-<pinref part="C4" gate="G$1" pin="1"/>
-<junction x="187.96" y="205.74"/>
 <junction x="195.58" y="185.42"/>
 <pinref part="J2" gate="G$1" pin="2"/>
@@
 <wire x1="215.9" y1="165.1" x2="215.9" y2="170.18" width="0.1524" layer="91"/>
 <junction x="215.9" y="170.18"/>
+<pinref part="C5" gate="G$1" pin="+"/>
+<junction x="187.96" y="205.74"/>
 </segment>
 </net>
@@
 </segment>
 </net>
-<net name="N$17" class="0">
+<net name="12V" class="0">
 <segment>
 <pinref part="IC1" gate="A1" pin="VI"/>
-<pinref part="C2" gate="G$1" pin="1"/>
 <wire x1="160.02" y1="205.74" x2="165.1" y2="205.74" width="0.1524" layer="91"/>
 <junction x="160.02" y="205.74"/>
@@
 <wire x1="287.02" y1="142.24" x2="276.86" y2="142.24" width="0.1524" layer="91"/>
 <junction x="276.86" y="142.24"/>
+<pinref part="C3" gate="G$1" pin="+"/>
 </segment>
 </net>
@@
 <net name="N$6" class="0">
 <segment>
-<pinref part="LED1" gate="G$1" pin="A"/>
 <pinref part="R2" gate="G$1" pin="2"/>
-<wire x1="294.64" y1="149.86" x2="289.56" y2="149.86" width="0.1524" layer="91"/>
-</segment>
-</net>
+<wire x1="293.37" y1="149.86" x2="289.56" y2="149.86" width="0.1524" layer="91"/>
+<pinref part="LED3" gate="G$1" pin="A"/>
+</segment>
+</net>

Commit message: Add files via upload
Connections:
- net 5V: now also U1.VCC; no longer R1.1
- net N$10: now also R1.2
- net N$2: now also R1.1; no longer R1.2, U1.VCC
- net N$9: now also U1.PC0
Other:
- moved on the sheet: R1, S1
Changed lines of the file:
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@@
 <instance part="GND3" gate="1" x="187.96" y="193.04"/>
 <instance part="GND4" gate="1" x="218.44" y="128.27" rot="MR0"/>
-<instance part="S1" gate="S" x="236.22" y="185.42" smashed="yes">
-<attribute name="NAME" x="234.95" y="180.34" size="1.778" layer="95"/>
-<attribute name="VALUE" x="226.06" y="193.04" size="1.778" layer="96"/>
-</instance>
-<instance part="GND6" gate="1" x="254" y="182.88"/>
+<instance part="S1" gate="S" x="179.07" y="97.79" smashed="yes">
+<attribute name="NAME" x="177.8" y="92.71" size="1.778" layer="95"/>
+<attribute name="VALUE" x="168.91" y="105.41" size="1.778" layer="96"/>
+</instance>
+<instance part="GND6" gate="1" x="190.5" y="86.36"/>
 <instance part="J1" gate="G$1" x="143.51" y="198.12"/>
 <instance part="GND7" gate="1" x="152.4" y="193.04"/>
@@
 <attribute name="VALUE" x="189.23" y="174.498" size="1.778" layer="96"/>
 </instance>
-<instance part="R1" gate="G$1" x="205.74" y="177.8" smashed="yes">
-<attribute name="NAME" x="204.47" y="180.5686" size="1.778" layer="95"/>
-<attribute name="VALUE" x="204.47" y="174.498" size="1.778" layer="96"/>
+<instance part="R1" gate="G$1" x="173.99" y="119.38" smashed="yes" rot="R90">
+<attribute name="NAME" x="171.2214" y="118.11" size="1.778" layer="95" rot="R90"/>
+<attribute name="VALUE" x="177.292" y="118.11" size="1.778" layer="96" rot="R90"/>
 </instance>
 <instance part="LED2" gate="G$1" x="185.42" y="170.18" smashed="yes">
@@
 <segment>
 <pinref part="S1" gate="S" pin="3"/>
-<wire x1="241.3" y1="185.42" x2="254" y2="185.42" width="0.1524" layer="91"/>
+<wire x1="184.15" y1="97.79" x2="190.5" y2="97.79" width="0.1524" layer="91"/>
+<wire x1="190.5" y1="97.79" x2="190.5" y2="88.9" width="0.1524" layer="91"/>
 <pinref part="GND6" gate="1" pin="GND"/>
 </segment>
@@
 <segment>
 <pinref part="S1" gate="S" pin="1"/>
-<wire x1="215.9" y1="177.8" x2="215.9" y2="185.42" width="0.1524" layer="91"/>
-<wire x1="215.9" y1="185.42" x2="231.14" y2="185.42" width="0.1524" layer="91"/>
-<wire x1="215.9" y1="177.8" x2="210.82" y2="177.8" width="0.1524" layer="91"/>
-<junction x="215.9" y="177.8"/>
-<pinref part="U1" gate="A" pin="VCC"/>
-<wire x1="215.9" y1="177.8" x2="215.9" y2="172.72" width="0.1524" layer="91"/>
-<wire x1="215.9" y1="172.72" x2="218.44" y2="172.72" width="0.1524" layer="91"/>
-<pinref part="R1" gate="G$1" pin="2"/>
+<pinref part="R1" gate="G$1" pin="1"/>
+<wire x1="173.99" y1="114.3" x2="173.99" y2="97.79" width="0.1524" layer="91"/>
 </segment>
 </net>
@@
 <segment>
 <pinref part="U1" gate="A" pin="PC6"/>
-<wire x1="144.78" y1="124.46" x2="254" y2="124.46" width="0.1524" layer="91"/>
+<wire x1="144.78" y1="124.46" x2="173.99" y2="124.46" width="0.1524" layer="91"/>
+<wire x1="173.99" y1="124.46" x2="254" y2="124.46" width="0.1524" layer="91"/>
 <wire x1="254" y1="124.46" x2="254" y2="134.62" width="0.1524" layer="91"/>
 <pinref part="J2" gate="G$1" pin="5"/>
 <wire x1="147.32" y1="160.02" x2="144.78" y2="160.02" width="0.1524" layer="91"/>
 <wire x1="144.78" y1="160.02" x2="144.78" y2="124.46" width="0.1524" layer="91"/>
+<pinref part="R1" gate="G$1" pin="2"/>
+<junction x="173.99" y="124.46"/>
 </segment>
 </net>
@@
 <wire x1="195.58" y1="205.74" x2="195.58" y2="185.42" width="0.1524" layer="91"/>
 <wire x1="195.58" y1="185.42" x2="195.58" y2="177.8" width="0.1524" layer="91"/>
-<wire x1="195.58" y1="170.18" x2="195.58" y2="177.8" width="0.1524" layer="91"/>
-<wire x1="200.66" y1="177.8" x2="195.58" y2="177.8" width="0.1524" layer="91"/>
+<wire x1="195.58" y1="170.18" x2="195.58" y2="172.72" width="0.1524" layer="91"/>
 <junction x="195.58" y="177.8"/>
 <pinref part="U1" gate="A" pin="AVCC"/>
+<wire x1="195.58" y1="172.72" x2="195.58" y2="177.8" width="0.1524" layer="91"/>
 <wire x1="218.44" y1="170.18" x2="215.9" y2="170.18" width="0.1524" layer="91"/>
 <pinref part="R3" gate="G$1" pin="2"/>
 <junction x="195.58" y="177.8"/>
-<pinref part="R1" gate="G$1" pin="1"/>
 <junction x="195.58" y="185.42"/>
 <pinref part="J2" gate="G$1" pin="2"/>
@@
 <pinref part="C5" gate="G$1" pin="+"/>
 <junction x="187.96" y="205.74"/>
+<pinref part="U1" gate="A" pin="VCC"/>
+<wire x1="218.44" y1="172.72" x2="195.58" y2="172.72" width="0.1524" layer="91"/>
+<junction x="195.58" y="172.72"/>
 </segment>
 </net>
@@
 <pinref part="R2" gate="G$1" pin="1"/>
 <wire x1="254" y1="149.86" x2="279.4" y2="149.86" width="0.1524" layer="91"/>
-</segment>
-</net>
+<pinref part="U1" gate="A" pin="PC0"/>
+</segment>
+</net>
